Commit message: fixed logo texture bug

File: rov_ricketts_description/urdf/base.xacro (robot description, xacro)
@@ -30,5 +30,5 @@
         <geometry>
           <mesh
-            filename="file://$(find rov_ricketts_description)/meshes/float.dae" scale="1.0 1.0 1.0"/>
+            filename="file://$(find rov_ricketts_description)/meshes/floatLogo.dae" scale="1.0 1.0 1.0"/>
         </geometry>
       </visual>
@@ -39,8 +39,8 @@
         <geometry>
           <mesh
-            filename="file://$(find rov_ricketts_description)/meshes/float.dae" scale="1.0 1.0 1.0"/>
+            filename="file://$(find rov_ricketts_description)/meshes/floatLogo.dae" scale="1.0 1.0 1.0"/>
         </geometry>
       </collision>
-      <visual>
+      <!-- <visual>
         <origin
           xyz="0 0 0"
@@ -50,4 +50,7 @@
             filename="file://$(find rov_ricketts_description)/meshes/decal.dae" scale="1.0 1.0 1.0"/>
         </geometry>
+        <material name="logo">
+          <texture filename="file://$(find rov_ricketts_description)/textures/logo.png"/>
+        </material>
       </visual>
       <collision>
@@ -59,5 +62,5 @@
             filename="file://$(find rov_ricketts_description)/meshes/decal.dae" scale="1.0 1.0 1.0"/>
         </geometry>
-      </collision>
+      </collision> -->
       <visual>
         <origin
