Commit message: Add Thrusters with Joint and Rviz Config
Color still to be fixed

File: rov_ricketts_description/urdf/Ricketts.xacro (robot description, xacro)
@@ -3,9 +3,31 @@
   <xacro:include filename="base.xacro" />
   <xacro:include filename="thrusters.xacro" />
-  <!-- Use macro to define base and thrusters -->
+  <!-- Use macro to define Base and Thrusters -->
   <link name="world"/>
+  <!-- Base -->
   <xacro:base_macro/>
-  <xacro:thruster_macro name="front_dx">
+  <!-- Front Thrusters -->
+  <xacro:thruster_macro name="front_sx">
              <origin xyz="-0.547848 0.4574 0.120838" rpy="${pi/4} ${pi/2} 0"/>
   </xacro:thruster_macro>
+  <xacro:thruster_macro name="front_dx">
+             <origin xyz="-0.547848 -0.4574 0.120838" rpy="${-pi/4} ${pi/2} 0"/>
+  </xacro:thruster_macro>
+  <!-- Back Thrusters -->
+  <xacro:thruster_macro name="rear_dx">
+             <origin xyz="-3.10256  -0.584898 0.121177" rpy="${-pi/2 -pi/4} ${pi/2} 0"/>
+  </xacro:thruster_macro>
+  <xacro:thruster_macro name="rear_sx">
+             <origin xyz="-3.10256   0.584898 0.121177" rpy="${pi/2 + pi/4} ${pi/2} 0"/>
+  </xacro:thruster_macro>
+   <!-- Up Thrusters -->
+  <xacro:thruster_macro name="up_rear">
+             <origin xyz="-3.10346   -0.000003 0.787413" rpy="0 0 0"/>
+  </xacro:thruster_macro>
+  <xacro:thruster_macro name="up_front_sx">
+             <origin xyz="-1.23346   0.652772  0.814842" rpy="${15/180 * pi} 0 0"/>
+  </xacro:thruster_macro>
+  <xacro:thruster_macro name="up_front_dx">
+             <origin xyz="-1.23346   -0.652772 0.814842" rpy="${-15/180 * pi} 0 0"/>
+  </xacro:thruster_macro>
 </robot>

File: rov_ricketts_description/urdf/base.xacro (robot description, xacro)
@@ -31,5 +31,5 @@
       </geometry>
       <material name="">
-        <color rgba="0.2 0.2 0.03 1" />
+        <color rgba="1 0.95 0.5 1" />
       </material>
     </visual>

File: rov_ricketts_description/urdf/thrusters.xacro (robot description, xacro)
@@ -38,5 +38,5 @@
           name="">
           <color
-            rgba="0.5 0.1 0.1 1" />
+            rgba="0.5 0.5 0.5 1" />
         </material>
       </visual>

Commit message: Correct texture
(conversions in Blender)
- using .dae instead of .stl for meshes
- .dae and texture .png in the same meshes folder due to dae information
- all base as single or multiple links

File: rov_ricketts_description/urdf/Ricketts.xacro (robot description, xacro)
@@ -2,8 +2,10 @@
 <robot name="Rov_Ricketts" xmlns:xacro="http://ros.org/wiki/xacro">
   <xacro:include filename="base.xacro" />
+  <xacro:include filename="base_separated.xacro" />
   <xacro:include filename="thrusters.xacro" />
   <!-- Use macro to define Base and Thrusters -->
   <link name="world"/>
   <!-- Base -->
+  <!-- <xacro:base_separated_macro/> -->
   <xacro:base_macro/>
   <!-- Front Thrusters -->

File: rov_ricketts_description/urdf/base.xacro (robot description, xacro)
@@ -2,4 +2,6 @@
 <robot xmlns:xacro="http://ros.org/wiki/xacro">
   <xacro:macro name="base_macro">
+  <!-- This macro is used to define robot body as unique links. This can be useful if you want to set a simple
+        approxiametd Inertia for the overall body -->
     <joint name="world_base_joint" type="fixed">
       <origin rpy="0 0 0" xyz="0 0 0"/>
@@ -8,40 +10,109 @@
     </joint>
     <link name="base_link">
-    <inertial>
-      <origin
-        xyz="0 0 0"
-        rpy="0 0 0" />
-      <mass
-        value="3.1152" />
-      <inertia
-        ixx="0.0036482"
-        ixy="7.8081E-07"
-        ixz="1.7521E-06"
-        iyy="0.0062179"
-        iyz="-1.4424E-06"
-        izz="0.0034682" />
-    </inertial>
-    <visual>
-      <origin
-        xyz="0 0 0"
-        rpy="0 0 0" />
-      <geometry>
-        <mesh
-          filename="file://$(find rov_ricketts_description)/meshes/body.stl" scale="1.0 1.0 1.0"/>
-      </geometry>
-      <material name="">
-        <color rgba="1 0.95 0.5 1" />
-      </material>
-    </visual>
-    <collision>
-      <origin
-        xyz="0 0 0"
-        rpy="0 0 0" />
-      <geometry>
-        <mesh
-          filename="file://$(find rov_ricketts_description)/meshes/body.stl" scale="1.0 1.0 1.0"/>
-      </geometry>
-    </collision>
-  </link>
+      <inertial>
+        <origin
+          xyz="0 0 0"
+          rpy="0 0 0" />
+        <mass
+          value="3.1152" />
+        <inertia
+          ixx="0.0036482"
+          ixy="7.8081E-07"
+          ixz="1.7521E-06"
+          iyy="0.0062179"
+          iyz="-1.4424E-06"
+          izz="0.0034682" />
+      </inertial>
+      <visual>
+        <origin
+          xyz="0 0 0"
+          rpy="0 0 0" />
+        <geometry>
+          <mesh
+            filename="file://$(find rov_ricketts_description)/meshes/float.dae" scale="1.0 1.0 1.0"/>
+        </geometry>
+      </visual>
+      <collision>
+        <origin
+          xyz="0 0 0"
+          rpy="0 0 0" />
+        <geometry>
+          <mesh
+            filename="file://$(find rov_ricketts_description)/meshes/float.dae" scale="1.0 1.0 1.0"/>
+        </geometry>
+      </collision>
+      <visual>
+        <origin
+          xyz="0 0 0"
+          rpy="0 0 0" />
+        <geometry>
+          <mesh
+            filename="file://$(find rov_ricketts_description)/meshes/decal.dae" scale="1.0 1.0 1.0"/>
+        </geometry>
+      </visual>
+      <collision>
+        <origin
+          xyz="0 0 0"
+          rpy="0 0 0" />
+        <geometry>
+          <mesh
+            filename="file://$(find rov_ricketts_description)/meshes/decal.dae" scale="1.0 1.0 1.0"/>
+        </geometry>
+      </collision>
+      <visual>
+        <origin
+          xyz="0 0 0"
+          rpy="0 0 0" />
+        <geometry>
+          <mesh
+            filename="file://$(find rov_ricketts_description)/meshes/frame.dae" scale="1.0 1.0 1.0"/>
+        </geometry>
+      </visual>
+      <collision>
+        <origin
+          xyz="0 0 0"
+          rpy="0 0 0" />
+        <geometry>
+          <mesh
+            filename="file://$(find rov_ricketts_description)/meshes/frame.dae" scale="1.0 1.0 1.0"/>
+        </geometry>
+      </collision>
+      <visual>
+        <origin
+          xyz="0 0 0"
+          rpy="0 0 0" />
+        <geometry>
+          <mesh
+            filename="file://$(find rov_ricketts_description)/meshes/thrusters.dae" scale="1.0 1.0 1.0"/>
+        </geometry>
+      </visual>
+      <collision>
+        <origin
+          xyz="0 0 0"
+          rpy="0 0 0" />
+        <geometry>
+          <mesh
+            filename="file://$(find rov_ricketts_description)/meshes/thrusters.dae" scale="1.0 1.0 1.0"/>
+        </geometry>
+      </collision>
+      <visual>
+        <origin
+          xyz="0 0 0"
+          rpy="0 0 0" />
+        <geometry>
+          <mesh
+            filename="file://$(find rov_ricketts_description)/meshes/equipment.dae" scale="1.0 1.0 1.0"/>
+        </geometry>
+      </visual>
+      <collision>
+        <origin
+          xyz="0 0 0"
+          rpy="0 0 0" />
+        <geometry>
+          <mesh
+            filename="file://$(find rov_ricketts_description)/meshes/equipment.dae" scale="1.0 1.0 1.0"/>
+        </geometry>
+      </collision>
+    </link>
   </xacro:macro>
 </robot>

File: rov_ricketts_description/urdf/thrusters.xacro (robot description, xacro)
@@ -33,5 +33,5 @@
         <geometry>
           <mesh
-            filename="file://$(find rov_ricketts_description)/meshes/thruster.stl" />
+            filename="file://$(find rov_ricketts_description)/meshes/propeller.stl" />
         </geometry>
         <material
@@ -45,5 +45,5 @@
         <geometry>
           <mesh
-            filename="file://$(find rov_ricketts_description)/meshes/thruster.stl" />
+            filename="file://$(find rov_ricketts_description)/meshes/propeller.stl" />
         </geometry>
       </collision>

Commit message: add arm base with revolute joint

File: rov_ricketts_description/urdf/Ricketts.xacro (robot description, xacro)
@@ -4,4 +4,5 @@
   <xacro:include filename="base_separated.xacro" />
   <xacro:include filename="thrusters.xacro" />
+  <xacro:include filename="arm.xacro" />
   <!-- Use macro to define Base and Thrusters -->
   <link name="world"/>
@@ -33,3 +34,6 @@
              <origin xyz="-1.23346   -0.652772 0.814842" rpy="${-15/180 * pi} 0 0"/>
   </xacro:thruster_macro>
+  <xacro:arm_macro name="arm">
+            <origin xyz="-0.291179 0.967229 ${-0.50857-0.1132}" rpy="0 0 0" />
+  </xacro:arm_macro>
 </robot>

File: rov_ricketts_description/urdf/arm.xacro (robot description, xacro)
@@ -1,9 +1,9 @@
 <?xml version="1.0" encoding="utf-8"?>
 <robot xmlns:xacro="http://ros.org/wiki/xacro">
-  <xacro:macro name="thruster_macro" params="name *origin">
-    <joint name="${name}_thruster" type="revolute">
+  <xacro:macro name="arm_macro" params="name *origin">
+    <joint name="${name}_base_joint" type="revolute">
       <xacro:insert_block name="origin"/>
       <parent link="base_link" />
-      <child link="${name}" />
+      <child link="${name}_base" />
       <axis xyz="0 0 1" />
       <limit
@@ -14,16 +14,5 @@
     </joint>
     <link
-      name="${name}">
-      <inertial>
-        <origin xyz="0 0 0" rpy="0 0 0" />
-        <mass value="0.12821" />
-        <inertia
-          ixx="3.7005E-05"
-          ixy="-1.9987E-08"
-          ixz="-3.8346E-12"
-          iyy="2.9934E-05"
-          iyz="2.5988E-11"
-          izz="4.8164E-05" />
-      </inertial>
+      name="${name}_base">
       <visual>
         <origin
@@ -32,5 +21,5 @@
         <geometry>
           <mesh
-            filename="file://$(find rov_ricketts_description)/meshes/propeller.stl" />
+            filename="file://$(find rov_ricketts_description)/meshes/arm_base.stl" />
         </geometry>
         <material
@@ -44,5 +33,5 @@
         <geometry>
           <mesh
-            filename="file://$(find rov_ricketts_description)/meshes/propeller.stl" />
+            filename="file://$(find rov_ricketts_description)/meshes/arm_base.stl" />
         </geometry>
       </collision>

Commit message: Add arm URDF Model and stl
Derived from sketchfab model, dividing and translating frames

File: rov_ricketts_description/urdf/Ricketts.xacro (robot description, xacro)
@@ -4,5 +4,4 @@
   <xacro:include filename="base_separated.xacro" />
   <xacro:include filename="thrusters.xacro" />
-  <xacro:include filename="arm.xacro" />
   <!-- Use macro to define Base and Thrusters -->
   <link name="world"/>
@@ -34,6 +33,11 @@
              <origin xyz="-1.23346   -0.652772 0.814842" rpy="${-15/180 * pi} 0 0"/>
   </xacro:thruster_macro>
-  <xacro:arm_macro name="arm">
-            <origin xyz="-0.291179 0.967229 ${-0.50857-0.1132}" rpy="0 0 0" />
-  </xacro:arm_macro>
+   <!-- Conditional Arm Loading, accordingly to launch argument -->
+  <xacro:arg name="load_arm" default="false" />
+  <xacro:if value="$(arg load_arm)">
+    <xacro:include filename="arm.xacro" />
+    <xacro:arm_macro name="arm">
+              <origin xyz="-0.291179 0.967229 ${-0.50857-0.1132}" rpy="0 0 0" />
+    </xacro:arm_macro>
+  </xacro:if>
 </robot>

File: rov_ricketts_description/urdf/arm.xacro (robot description, xacro)
@@ -37,4 +37,235 @@
       </collision>
     </link>
+    <joint name="${name}_base_link1" type="revolute">
+      <origin
+          xyz="0.122041  -0.036335   0.175604 "
+          rpy="0 0 -0.3106" />
+      <parent link="${name}_base" />
+      <child link="${name}_link1" />
+      <axis xyz="0 1 0" />
+      <limit
+        lower="-3.14"
+        upper="3.14"
+        effort="20"
+        velocity="10" />
+    </joint>
+    <link
+      name="${name}_link1">
+      <visual>
+        <origin
+          xyz="0 0 0"
+          rpy="0 0 0" />
+        <geometry>
+          <mesh
+            filename="file://$(find rov_ricketts_description)/meshes/arm_link1.stl" />
+        </geometry>
+        <material
+          name="">
+          <color
+            rgba="0.5 0.5 0.5 1" />
+        </material>
+      </visual>
+      <collision>
+        <origin xyz="0 0 0" rpy="0 0 0" />
+        <geometry>
+          <mesh
+            filename="file://$(find rov_ricketts_description)/meshes/arm_link1.stl" />
+        </geometry>
+      </collision>
+    </link>
+    <joint name="${name}_link1_link2" type="revolute">
+      <origin
+          xyz="  0.2440 0.0  0.815517 "
+          rpy="0 0 0" />
+      <parent link="${name}_link1" />
+      <child link="${name}_link2" />
+      <axis xyz="0 1 0" />
+      <limit
+        lower="-3.14"
+        upper="3.14"
+        effort="20"
+        velocity="10" />
+    </joint>
+    <link
+      name="${name}_link2">
+      <visual>
+        <origin
+          xyz="0 0 0"
+          rpy="0 0 0" />
+        <geometry>
+          <mesh
+            filename="file://$(find rov_ricketts_description)/meshes/arm_link2.stl" />
+        </geometry>
+        <material
+          name="">
+          <color
+            rgba="0.5 0.5 0.5 1" />
+        </material>
+      </visual>
+      <collision>
+        <origin xyz="0 0 0" rpy="0 0 0" />
+        <geometry>
+          <mesh
+            filename="file://$(find rov_ricketts_description)/meshes/arm_link2.stl" />
+        </geometry>
+      </collision>
+    </link>
+    <joint name="${name}_link2_link3" type="revolute">
+      <origin
+          xyz="  0.2268 0.0 -0.425988  "
+          rpy="0 0 0" />
+      <parent link="${name}_link2" />
+      <child link="${name}_link3" />
+      <axis xyz="0 1 0" />
+      <limit
+        lower="-3.14"
+        upper="3.14"
+        effort="20"
+        velocity="10" />
+    </joint>
+    <link
+      name="${name}_link3">
+      <visual>
+        <origin
+          xyz="0 0 0"
+          rpy="0 0 0" />
+        <geometry>
+          <mesh
+            filename="file://$(find rov_ricketts_description)/meshes/arm_link3.stl" />
+        </geometry>
+        <material
+          name="">
+          <color
+            rgba="0.5 0.5 0.5 1" />
+        </material>
+      </visual>
+      <collision>
+        <origin xyz="0 0 0" rpy="0 0 0" />
+        <geometry>
+          <mesh
+            filename="file://$(find rov_ricketts_description)/meshes/arm_link3.stl" />
+        </geometry>
+      </collision>
+    </link>
+    <joint name="${name}_link3_link4" type="revolute">
+      <origin
+          xyz=" 0.017629 0 -0.170456"
+          rpy="0 ${pi - 0.0952} 0" />
+      <parent link="${name}_link3" />
+      <child link="${name}_link4" />
+      <axis xyz="0  0 1" />
+      <limit
+        lower="-3.14"
+        upper="3.14"
+        effort="20"
+        velocity="10" />
+    </joint>
+    <link
+      name="${name}_link4">
+      <visual>
+        <origin
+          xyz="0 0 0"
+          rpy="0 0 0" />
+        <geometry>
+          <mesh
+            filename="file://$(find rov_ricketts_description)/meshes/arm_link4.stl" />
+        </geometry>
+        <material
+          name="">
+          <color
+            rgba="0.5 0.5 0.5 1" />
+        </material>
+      </visual>
+      <collision>
+        <origin xyz="0 0 0" rpy="0 0 0" />
+        <geometry>
+          <mesh
+            filename="file://$(find rov_ricketts_description)/meshes/arm_link4.stl" />
+        </geometry>
+      </collision>
+    </link>
+    <joint name="${name}_link4_claw_right" type="revolute">
+      <origin
+          xyz=" 0.0042 -0.0328 0.14"
+          rpy="0 0 0" />
+      <parent link="${name}_link4" />
+      <child link="${name}_claw_right" />
+      <axis xyz="1 0 0" />
+      <limit
+        lower="-3.14"
+        upper="3.14"
+        effort="20"
+        velocity="10" />
+    </joint>
+    <link
+      name="${name}_claw_right">
+      <visual>
+        <origin
+          xyz="0 0 0"
+          rpy="0 0 0" />
+        <geometry>
+          <mesh
+            filename="file://$(find rov_ricketts_description)/meshes/grip_claw.stl" />
+        </geometry>
+        <material
+          name="">
+          <color
+            rgba="0.5 0.5 0.5 1" />
+        </material>
+      </visual>
+      <collision>
+        <origin xyz="0 0 0" rpy="0 0 0" />
+        <geometry>
+          <mesh
+            filename="file://$(find rov_ricketts_description)/meshes/grip_claw.stl" />
+        </geometry>
+      </collision>
+    </link>
+    <joint name="${name}_link4_claw_left" type="revolute">
+      <mimic joint="${name}_link4_claw_right" multiplier="1" offset="0"/>
+      <origin
+          xyz=" 0.0042 0.0328 0.14"
+          rpy="0 0 ${pi}" />
+      <parent link="${name}_link4" />
+      <child link="${name}_claw_left" />
+      <axis xyz="1 0 0" />
+      <limit
+        lower="-3.14"
+        upper="3.14"
+        effort="20"
+        velocity="10" />
+    </joint>
+    <link
+      name="${name}_claw_left">
+      <visual>
+        <origin
+          xyz="0 0 0"
+          rpy="0 0 0" />
+        <geometry>
+          <mesh
+            filename="file://$(find rov_ricketts_description)/meshes/grip_claw.stl" />
+        </geometry>
+        <material
+          name="">
+          <color
+            rgba="0.5 0.5 0.5 1" />
+        </material>
+      </visual>
+      <collision>
+        <origin xyz="0 0 0" rpy="0 0 0" />
+        <geometry>
+          <mesh
+            filename="file://$(find rov_ricketts_description)/meshes/grip_claw.stl" />
+        </geometry>
+      </collision>
+    </link>
+    <joint name="${name}_hand_tool" type="fixed">
+      <origin
+          xyz=" 0 0  0.271942"
+          rpy="0 0 ${pi}" />
+      <parent link="${name}_link4" />
+      <child link="${name}_tool" />
+    </joint>
+    <link name="${name}_tool" />
   </xacro:macro>
 </robot>
