Commit message: tentative to fix buoyancy...
Plugin studied but behavior still not as expected

File: rov_ricketts_description/urdf/base_separate_float.xacro (robot description, xacro)
@@ -7,15 +7,15 @@
       <inertial>
         <origin
-          xyz="-1.81450712  0.00636514  0.5734822"
+          xyz="-1.71648272  0.02593398 -0.13442244"
           rpy="0 0 0" />
         <mass
-          value="4700.0" />
+          value="4000.0" />
         <inertia
-          ixx="2779.72167757"
-          ixy="-142.69321245"
-          ixz="-59.10699454"
-          iyy="4409.88731132"
-          iyz="31.89417598"
-          izz="4961.49762669" />
+          ixx="3136.45125968"
+          ixy="-486.35412743"
+          ixz="-536.21655801"
+          iyy="3051.79345927"
+          iyz="37.63656271"
+          izz="4598.19910255" />
       </inertial>
       <!-- <inertial>
@@ -33,5 +33,5 @@
           izz="1E-2" />
       </inertial> -->
-      <visual>
+      <!-- <visual>
         <origin
           xyz="0 0 0"
@@ -49,4 +49,22 @@
           <mesh
             filename="file://$(find rov_ricketts_description)/meshes/floatLogo.dae" scale="1.0 1.0 1.0"/>
+        </geometry>
+      </collision> -->
+      <visual>
+        <origin
+          xyz="0 0 0"
+          rpy="0 0 0" />
+        <geometry>
+          <mesh
+            filename="file://$(find rov_ricketts_description)/meshes/frame.dae" scale="1.0 1.0 1.0"/>
+        </geometry>
+      </visual>
+      <collision>
+        <origin
+          xyz="0 0 0"
+          rpy="0 0 0" />
+        <geometry>
+          <mesh
+            filename="file://$(find rov_ricketts_description)/meshes/frame.dae" scale="1.0 1.0 1.0"/>
         </geometry>
       </collision>
@@ -72,22 +90,4 @@
         </geometry>
       </collision> -->
-      <visual>
-        <origin
-          xyz="0 0 0"
-          rpy="0 0 0" />
-        <geometry>
-          <mesh
-            filename="file://$(find rov_ricketts_description)/meshes/frame.dae" scale="1.0 1.0 1.0"/>
-        </geometry>
-      </visual>
-      <collision>
-        <origin
-          xyz="0 0 0"
-          rpy="0 0 0" />
-        <geometry>
-          <mesh
-            filename="file://$(find rov_ricketts_description)/meshes/frame.dae" scale="1.0 1.0 1.0"/>
-        </geometry>
-      </collision>
       <visual>
         <origin
@@ -126,5 +126,5 @@
         </geometry>
       </collision>
-    </link>
+     </link>
     <joint name="base_link_frame" type="fixed">
       <origin rpy="0 0 0" xyz="0 0 0"/>
@@ -148,4 +148,43 @@
       </inertial> -->
     </link>
+    <joint name="base_float_joint" type="fixed">
+      <origin rpy="0 0 0" xyz="-1.84651 0 0.798725"/>
+      <parent link="base_link" />
+      <child link="float_link" />
+    </joint>
+    <link name="float_link">
+      <inertial>
+        <origin
+          xyz="0 0 0"
+          rpy="0 0 0" />
+        <mass
+          value="700.0" />
+        <inertia
+          ixx="2.25940928E+02"
+          ixy="-8.14319126E-03"
+          ixz="-2.52907176E+00"
+          iyy="5.49374390E+02"
+          iyz="1.50415351E-04"
+          izz="7.14667057E+02" />
+      </inertial>
+      <visual>
+        <origin
+          xyz="1.84651 0 -0.798725"
+          rpy="0 0 0" />
+        <geometry>
+          <mesh
+            filename="file://$(find rov_ricketts_description)/meshes/floatLogo2.dae" scale="1.0 1.0 1.0"/>
+        </geometry>
+      </visual>
+      <collision>
+        <origin
+          xyz="1.84651 0 -0.798725"
+          rpy="0 0 0" />
+        <geometry>
+          <mesh
+            filename="file://$(find rov_ricketts_description)/meshes/floatLogo2.dae" scale="1.0 1.0 1.0"/>
+        </geometry>
+      </collision>
+    </link>
 <!--
     <joint name="base_sonar_joint" type="fixed">

File: rov_ricketts_description/urdf/gazebo_physics.xacro (robot description, xacro)
@@ -7,9 +7,14 @@
         <link_name>base_link</link_name>
         <namespace>rov_ricketts</namespace>
-        <min_volume>-60.0</min_volume>
-        <neutral_volume>0</neutral_volume>
-        <default_volume>-30.0</default_volume>
-        <max_volume>60.0</max_volume>
-        <max_inflation_rate>0.5</max_inflation_rate>
+        <min_volume>-30.0</min_volume>
+        <neutral_volume>4.7</neutral_volume>
+        <default_volume>-25.0</default_volume>
+        <max_volume>30.0</max_volume>
+        <surface>0.0</surface>
+        <max_inflation_rate>2.5</max_inflation_rate>
+      </plugin>
+      <plugin
+            filename="gz-sim-odometry-publisher-system"
+            name="gz::sim::systems::OdometryPublisher">
       </plugin>
     </gazebo>

File: rov_ricketts_description/urdf/joint_states_plugin.xacro (robot description, xacro)
@@ -8,4 +8,5 @@
                 <!-- <update_rate>500</update_rate> -->
                 <topic>/joint_states</topic>
+                <!-- <joint_name>base_float_joint</joint_name> -->
                 <joint_name>front_sx_thruster</joint_name>
                 <joint_name>front_dx_thruster</joint_name>
