Commit message: controlling  thrusters but not moving

File: rov_ricketts_description/urdf/thrusters.xacro (robot description, xacro)
@@ -2,12 +2,14 @@
 <robot xmlns:xacro="http://ros.org/wiki/xacro">
   <xacro:macro name="thruster_macro" params="name *origin">
-    <joint name="${name}_thruster" type="continuous">
+    <joint name="${name}_thruster" type="revolute">
       <xacro:insert_block name="origin"/>
       <parent link="base_frame" />
       <child link="${name}" />
-      <axis xyz="0 0 1" />
-      <limit
-        effort="1E12"
-        velocity="200" />
+        <axis xyz="0 0 1" />
+        <limit
+          lower="-1E12"
+          upper="1E12"
+          effort="1E6"
+          velocity="100" />
     </joint>
     <link
@@ -52,5 +54,6 @@
         name="gz::sim::systems::Thruster">
         <joint_name>${name}_thruster</joint_name>
-        <thrust_coefficient>0.004</thrust_coefficient>
+        <namespace>rov_ricketts</namespace>
+        <thrust_coefficient>0.05</thrust_coefficient>
         <fluid_density>1000</fluid_density>
         <propeller_diameter>0.38</propeller_diameter>
