Commit message: add  missing inertia and joint Plugins

File: rov_ricketts_description/urdf/Ricketts.urdf.xacro (robot description, xacro)
@@ -4,4 +4,5 @@
   <xacro:include filename="base_separated.xacro" />
   <xacro:include filename="thrusters.xacro" />
+  <xacro:include filename="thrusters_joint_states_plugin.xacro" />
   <!-- Use macro to define Base and Thrusters -->
   <link name="world"/>
@@ -37,7 +38,9 @@
   <xacro:if value="$(arg load_arm)">
     <xacro:include filename="arm.xacro" />
+    <xacro:include filename="arm_joint_states_plugin.xacro" />
     <xacro:arm_macro name="arm">
               <origin xyz="-0.291179 0.967229 ${-0.50857-0.1132}" rpy="0 0 0" />
     </xacro:arm_macro>
+    <xacro:joint_state_macro name="arm"/>
   </xacro:if>
 </robot>

File: rov_ricketts_description/urdf/arm.xacro (robot description, xacro)
@@ -304,5 +304,5 @@
       </collision>
     </link>
-    <joint name="${name}_link4_claw_right" type="revolute">
+    <joint name="${name}_link5_claw_right" type="revolute">
       <origin
           xyz=" 0.0042 -0.0328 0.14"
@@ -355,6 +355,6 @@
       </collision>
     </link>
-    <joint name="${name}_link4_claw_left" type="revolute">
-      <mimic joint="${name}_link4_claw_right" multiplier="1" offset="0"/>
+    <joint name="${name}_link5_claw_left" type="revolute">
+      <mimic joint="${name}_link5_claw_right" multiplier="1" offset="0"/>
       <origin
           xyz=" 0.0042 0.0328 0.14"

File: rov_ricketts_description/urdf/base.xacro (robot description, xacro)
@@ -12,15 +12,15 @@
       <inertial>
         <origin
-          xyz="0 0 0"
+          xyz="-1.81450712  0.00636514  0.5734822"
           rpy="0 0 0" />
         <mass
-          value="3.1152" />
+          value="4700.0" />
         <inertia
-          ixx="0.0036482"
-          ixy="7.8081E-07"
-          ixz="1.7521E-06"
-          iyy="0.0062179"
-          iyz="-1.4424E-06"
-          izz="0.0034682" />
+          ixx="2779.72167757"
+          ixy="-142.69321245"
+          ixz="-59.10699454"
+          iyy="4409.88731132"
+          iyz="31.89417598"
+          izz="4961.49762669" />
       </inertial>
       <visual>

File: rov_ricketts_description/urdf/thrusters.xacro (robot description, xacro)
@@ -13,15 +13,16 @@
     <link
       name="${name}">
-      <!-- <inertial>
-        <origin xyz="0 0 0" rpy="0 0 0" />
-        <mass value="0.12821" />
+      <inertial>
+        <origin xyz="1.29123983e-04 -4.30643335e-05  6.65557479e-04"
+                rpy="0 0 0" />
+        <mass value="2.8201033788020022" />
         <inertia
-          ixx="3.7005E-05"
-          ixy="-1.9987E-08"
-          ixz="-3.8346E-12"
-          iyy="2.9934E-05"
-          iyz="2.5988E-11"
-          izz="4.8164E-05" />
-      </inertial> -->
+          ixx="1.36253391E-02"
+          ixy="-3.62214961E-07"
+          ixz="-6.16491988E-07"
+          iyy="1.36232618E-02"
+          iyz="-9.76544753E-06"
+          izz="2.52722006E-02" />
+      </inertial>
       <visual>
         <origin

Commit message: fix URDF errors to load joints of arm

File: rov_ricketts_description/urdf/Ricketts.urdf.xacro (robot description, xacro)
@@ -4,4 +4,5 @@
   <xacro:include filename="base_separated.xacro" />
   <xacro:include filename="thrusters.xacro" />
+  <xacro:include filename="joint_states_plugin.xacro" />
   <!-- <xacro:include filename="thrusters_joint_states_plugin.xacro" />  -->
   <!-- Use macro to define Base and Thrusters -->
@@ -38,10 +39,9 @@
   <xacro:if value="$(arg load_arm)">
     <xacro:include filename="arm.xacro" />
-    <!-- <xacro:include filename="arm_joint_states_plugin.xacro" /> -->
     <xacro:arm_macro name="arm">
               <origin xyz="-0.291179 0.967229 ${-0.50857-0.1132}" rpy="0 0 0" />
     </xacro:arm_macro>
-    <xacro:joint_state_macro name="arm"/>
+    <!-- <xacro:joint_state_macro name="arm"/> -->
   </xacro:if>
-  <xacro:include filename="joint_states_plugin.xacro" />
+  <xacro:all_joint_state_macro load_arm = "load_arm" name="arm"/>
 </robot>

File: rov_ricketts_description/urdf/joint_states_plugin.xacro (robot description, xacro)
@@ -1,27 +1,30 @@
 <?xml version="1.0"?>
 <robot xmlns:xacro="http://ros.org/wiki/xacro">
-        <xacro:arg name="load_arm" default="false" />
+    <xacro:arg name="load_arm" default="false" />
+        <xacro:macro name="all_joint_state_macro" params="load_arm name">
             <!-- Gazebo plugin for joint state publisher  -->
-        <gazebo>
-            <plugin name="gz::sim::systems::JointStatePublisher" filename="gz-sim-joint-state-publisher-system">
-            <!-- <update_rate>500</update_rate> -->
-            <topic>/joint_states</topic>
-            <joint_name>front_sx_thruster</joint_name>
-            <joint_name>front_dx_thruster</joint_name>
-            <joint_name>rear_dx_thruster</joint_name>
-            <joint_name>rear_sx_thruster</joint_name>
-            <joint_name>up_rear_thruster</joint_name>
-            <joint_name>up_front_sx_thruster</joint_name>
-            <joint_name>up_front_dx_thruster</joint_name>
-            <xacro:if value="$(arg load_arm)">
-                <joint_name>${name}_base_link1</joint_name>
-                <joint_name>${name}_link1_link2</joint_name>
-                <joint_name>${name}_link2_link3</joint_name>
-                <joint_name>${name}_link3_link4</joint_name>
-                <joint_name>${name}_link4_link5</joint_name>
-                <joint_name>${name}_link5_claw_right</joint_name>
-                <joint_name>${name}_link5_claw_left</joint_name>
-            </xacro:if>
-            </plugin>
-        </gazebo>
+            <gazebo>
+                <plugin name="gz::sim::systems::JointStatePublisher" filename="gz-sim-joint-state-publisher-system">
+                <!-- <update_rate>500</update_rate> -->
+                <topic>/joint_states</topic>
+                <joint_name>front_sx_thruster</joint_name>
+                <joint_name>front_dx_thruster</joint_name>
+                <joint_name>rear_dx_thruster</joint_name>
+                <joint_name>rear_sx_thruster</joint_name>
+                <joint_name>up_rear_thruster</joint_name>
+                <joint_name>up_front_sx_thruster</joint_name>
+                <joint_name>up_front_dx_thruster</joint_name>
+                <xacro:if value="$(arg load_arm)">
+                    <joint_name>${name}_base_joint</joint_name>
+                    <joint_name>${name}_base_link1</joint_name>
+                    <joint_name>${name}_link1_link2</joint_name>
+                    <joint_name>${name}_link2_link3</joint_name>
+                    <joint_name>${name}_link3_link4</joint_name>
+                    <joint_name>${name}_link4_link5</joint_name>
+                    <joint_name>${name}_link5_claw_right</joint_name>
+                    <joint_name>${name}_link5_claw_left</joint_name>
+                </xacro:if>
+                </plugin>
+            </gazebo>
+        </xacro:macro>
 </robot>

Commit message: Buoyancy, Thrust and Sensors
WIP,  not working for now.
When buoyancy/volume is at -24.0 it starts to behave badly and sinks from the front! probaby because of how base link is positioned (in front). Try to position it on the CoM of the system

File: rov_ricketts_description/urdf/Ricketts.urdf.xacro (robot description, xacro)
@@ -5,7 +5,8 @@
   <xacro:include filename="thrusters.xacro" />
   <xacro:include filename="joint_states_plugin.xacro" />
+  <xacro:include filename="gazebo_physics.xacro" />
+  <xacro:include filename="sensors_plugins.xacro" />
   <!-- <xacro:include filename="thrusters_joint_states_plugin.xacro" />  -->
   <!-- Use macro to define Base and Thrusters -->
-  <link name="world"/>
   <!-- Base -->
   <!-- <xacro:base_separated_macro/> -->

File: rov_ricketts_description/urdf/base.xacro (robot description, xacro)
@@ -4,9 +4,4 @@
   <!-- This macro is used to define robot body as unique links. This can be useful if you want to set a simple
         approxiametd Inertia for the overall body -->
-    <joint name="world_base_joint" type="fixed">
-      <origin rpy="0 0 0" xyz="0 0 0"/>
-      <parent link="world" />
-      <child link="base_link" />
-    </joint>
     <link name="base_link">
       <inertial>
@@ -24,4 +19,18 @@
           izz="4961.49762669" />
       </inertial>
+      <!-- <inertial>
+        <origin
+          xyz="-1.81450712  0.00636514  0.5734822"
+          rpy="0 0 0" />
+        <mass
+          value="0.1" />
+        <inertia
+          ixx="1E-2"
+          ixy="0"
+          ixz="0"
+          iyy="1E-2"
+          iyz="0"
+          izz="1E-2" />
+      </inertial> -->
       <visual>
         <origin
@@ -118,4 +127,32 @@
       </collision>
     </link>
+      <joint name="base_link_frame" type="fixed">
+      <origin rpy="0 0 0" xyz="0 0 0"/>
+      <parent link="base_link" />
+      <child link="base_frame" />
+    </joint>
+    <link name="base_frame">
+      <!-- <inertial>
+        <origin
+          xyz="-1.81450712  0.00636514  0.5734822"
+          rpy="0 0 0" />
+        <mass
+          value="4700.0" />
+        <inertia
+          ixx="2779.72167757"
+          ixy="-142.69321245"
+          ixz="-59.10699454"
+          iyy="4409.88731132"
+          iyz="31.89417598"
+          izz="4961.49762669" />
+      </inertial> -->
+    </link>
+<!--
+    <joint name="base_sonar_joint" type="fixed">
+      <origin rpy="0 0 0"
+              xyz="-0.26829 -0.00011 1.29141"/>
+      <parent link="base_link" />
+      <child link="sonar_link" />
+    </joint> -->
   </xacro:macro>
 </robot>

File: rov_ricketts_description/urdf/thrusters.xacro (robot description, xacro)
@@ -4,10 +4,10 @@
     <joint name="${name}_thruster" type="continuous">
       <xacro:insert_block name="origin"/>
-      <parent link="base_link" />
+      <parent link="base_frame" />
       <child link="${name}" />
       <axis xyz="0 0 1" />
       <limit
-        effort="20"
-        velocity="10" />
+        effort="1E12"
+        velocity="200" />
     </joint>
     <link
@@ -47,4 +47,16 @@
       </collision>
     </link>
+    <gazebo>
+      <plugin
+        filename="gz-sim-thruster-system"
+        name="gz::sim::systems::Thruster">
+        <joint_name>${name}_thruster</joint_name>
+        <thrust_coefficient>0.004</thrust_coefficient>
+        <fluid_density>1000</fluid_density>
+        <propeller_diameter>0.38</propeller_diameter>
+        <max_thrust_cmd>10000</max_thrust_cmd>
+        <min_thrust_cmd>0</min_thrust_cmd>
+      </plugin>
+    </gazebo>
   </xacro:macro>
 </robot>

Commit message: new simulation world

File: rov_ricketts_description/urdf/Ricketts.urdf.xacro (robot description, xacro)
@@ -42,5 +42,5 @@
     <xacro:include filename="arm.xacro" />
     <xacro:arm_macro name="arm">
-              <origin xyz="-0.291179 0.967229 ${-0.50857-0.1132}" rpy="0 0 0" />
+              <origin xyz="${-0.291179+1.8143} ${0.967229-0.004215} ${-0.50857-0.1132-0.560595}" rpy="0 0 0" />
     </xacro:arm_macro>
     <!-- <xacro:joint_state_macro name="arm"/> -->

File: rov_ricketts_description/urdf/base_inertia_new.xacro (robot description, xacro)
@@ -85,4 +85,25 @@
       </inertial> -->
     </link>
+    <joint name="base_sonar_frame" type="fixed">
+      <origin rpy="0 0 0" xyz="1.54601 -0.004325 0.730815"/>
+      <parent link="base_link" />
+      <child link="sonar_frame" />
+    </joint>
+    <link name="sonar_frame">
+      <inertial>
+        <origin
+          xyz="0 0 0"
+          rpy="0 0 0" />
+        <mass
+          value="0.00000001" />
+        <inertia
+          ixx="1e-12"
+          ixy="0"
+          ixz="0"
+          iyy="1e-12"
+          iyz="0"
+          izz="1e-12" />
+      </inertial>
+    </link>
 <!--
     <joint name="base_sonar_joint" type="fixed">

File: rov_ricketts_description/urdf/gazebo_physics.xacro (robot description, xacro)
@@ -9,5 +9,5 @@
         <min_volume>-30.0</min_volume>
         <neutral_volume>4.7</neutral_volume>
-        <default_volume>-9.4</default_volume>
+        <default_volume>-5.8</default_volume>
         <max_volume>30.0</max_volume>
         <surface>1.0</surface>

File: rov_ricketts_description/urdf/sensors_plugins.xacro (robot description, xacro)
@@ -1,21 +1,22 @@
 <?xml version="1.0"?>
 <robot xmlns:xacro="http://ros.org/wiki/xacro">
-    <gazebo reference="base_link">
+    <gazebo reference="sonar_frame">
         <sensor name="sonar" type="gpu_ray">
-          <pose>-0.26829 -0.00011 1.29141 0 0 0</pose>
-          <update_rate>10</update_rate>
+          <!-- <pose>1.54601 -0.004325 0.730815 0 0 0</pose> -->
+          <pose>0 0 0 0 0 0</pose>
+          <update_rate>5</update_rate>
           <topic>sonar</topic>
           <ray>
             <scan>
               <horizontal>
-                <samples>1875</samples>
+                <samples>100</samples>
                 <resolution>1</resolution>
-                <min_angle>-3.1415926535897931</min_angle>
-                <max_angle>3.1415926535897931</max_angle>
+                <min_angle>-1.57</min_angle>
+                <max_angle>1.57</max_angle>
               </horizontal>
               <vertical>
-                <samples>16</samples>
+                <samples>20</samples>
                 <resolution>1</resolution>
-                <min_angle>0</min_angle>
+                <min_angle>-0.76</min_angle>
                 <max_angle>1.57</max_angle>
               </vertical>

File: rov_ricketts_description/urdf/thrusters.xacro (robot description, xacro)
@@ -59,5 +59,5 @@
         <propeller_diameter>0.38</propeller_diameter>
         <max_thrust_cmd>10000</max_thrust_cmd>
-        <min_thrust_cmd>0</min_thrust_cmd>
+        <min_thrust_cmd>-10000</min_thrust_cmd>
       </plugin>
     </gazebo>
