Commit message: clean up xacro description
- removed useless file
- conditional base inertia
- implemented simple inertia macro

File: rov_ricketts_description/urdf/Ricketts.urdf.xacro (robot description, xacro)
@@ -1,16 +1,25 @@
 <?xml version="1.0" encoding="utf-8"?>
 <robot name="Rov_Ricketts" xmlns:xacro="http://ros.org/wiki/xacro">
-  <!-- <xacro:include filename="base.xacro" /> -->
-  <xacro:include filename="base_inertia_new.xacro" />
+  <xacro:include filename="base.xacro" />
   <xacro:include filename="base_separated.xacro" />
   <xacro:include filename="thrusters.xacro" />
-  <xacro:include filename="joint_states_plugin.xacro" />
+  <xacro:include filename="joint_states_publisher_plugin.xacro" />
+  <!-- Set of macros for simple geometrical inertia: box, cylinder, sphere -->
+  <xacro:include filename="simple_inertial_macro.xacro" />
+  <!-- Load sensors: Sonar,... -->
+  <xacro:include filename="sensors_plugins.xacro" />
+  <!-- Load physics: Buoyancy,... -->
   <xacro:include filename="gazebo_physics.xacro" />
-  <xacro:include filename="sensors_plugins.xacro" />
-  <!-- <xacro:include filename="thrusters_joint_states_plugin.xacro" />  -->
-  <!-- Use macro to define Base and Thrusters -->
+  <!-- Use macro to define Base -->
   <!-- Base -->
   <!-- <xacro:base_separated_macro/> -->
-  <xacro:base_macro/>
+  <xacro:arg name="simple_inertia" default="false" />
+  <xacro:if value="$(arg simple_inertia)">
+    <xacro:base_macro simple_inertia="true"/>
+  </xacro:if>
+  <xacro:unless value="$(arg simple_inertia)">
+    <xacro:base_macro simple_inertia="false"/>
+  </xacro:unless>
+  <!-- Use macro to define Thrusters: front_sx, front_dx, rear_dx, rear_sx, up_rear, up_front_sx, up_front_dx -->
   <!-- Front Thrusters -->
   <xacro:thruster_macro name="front_sx">
@@ -44,6 +53,6 @@
               <origin xyz="${-0.291179+1.8143} ${0.967229-0.004215} ${-0.50857-0.1132-0.560595}" rpy="0 0 0" />
     </xacro:arm_macro>
-    <!-- <xacro:joint_state_macro name="arm"/> -->
   </xacro:if>
-  <xacro:all_joint_state_macro load_arm = "load_arm" name="arm"/>
+  <!-- Load joint state publisher gazebo plugin -->
+  <xacro:joint_states_publisher_macro load_arm="load_arm" name="arm"/>
 </robot>

File: rov_ricketts_description/urdf/base.xacro (robot description, xacro)
@@ -1,39 +1,33 @@
 <?xml version="1.0" encoding="utf-8"?>
 <robot xmlns:xacro="http://ros.org/wiki/xacro">
-  <xacro:macro name="base_macro">
+  <xacro:macro name="base_macro" params="simple_inertia">
   <!-- This macro is used to define robot body as unique links. This can be useful if you want to set a simple
         approxiametd Inertia for the overall body -->
     <link name="base_link">
-      <inertial>
-        <origin
-          xyz="-1.81450712  0.00636514  0.5734822"
-          rpy="0 0 0" />
-        <mass
-          value="4700.0" />
-        <inertia
-          ixx="2779.72167757"
-          ixy="-142.69321245"
-          ixz="-59.10699454"
-          iyy="4409.88731132"
-          iyz="31.89417598"
-          izz="4961.49762669" />
-      </inertial>
-      <!-- <inertial>
-        <origin
-          xyz="-1.81450712  0.00636514  0.5734822"
-          rpy="0 0 0" />
-        <mass
-          value="0.1" />
-        <inertia
-          ixx="1E-2"
-          ixy="0"
-          ixz="0"
-          iyy="1E-2"
-          iyz="0"
-          izz="1E-2" />
-      </inertial> -->
+      <xacro:if value="$(arg simple_inertia)">
+        <xacro:inertial_box mass="4700.0" x="3.3" y="1.80" z="1.80">
+              <origin xyz="0.0 0.0 -0.5" rpy="0 0 0"/>
+        </xacro:inertial_box>
+      </xacro:if>
+      <xacro:unless value="$(arg simple_inertia)">
+        <inertial>
+          <origin
+            xyz="0.0 0.0 -0.5"
+            rpy="0 0 0" />
+          <mass
+            value="4700.0" />
+          <inertia
+            ixx="2779.72167757"
+            ixy="-142.69321245"
+            ixz="-59.10699454"
+            iyy="4409.88731132"
+            iyz="31.89417598"
+            izz="4961.49762669" />
+        </inertial>
+      </xacro:unless>
+      <!-- float frame + side logo panel -->
       <visual>
         <origin
-          xyz="0 0 0"
+          xyz="1.8143 -0.004215 -0.560595"
           rpy="0 0 0" />
         <geometry>
@@ -42,37 +36,8 @@
         </geometry>
       </visual>
-      <collision>
-        <origin
-          xyz="0 0 0"
-          rpy="0 0 0" />
-        <geometry>
-          <mesh
-            filename="file://$(find rov_ricketts_description)/meshes/floatLogo.dae" scale="1.0 1.0 1.0"/>
-        </geometry>
-      </collision>
-      <!-- <visual>
-        <origin
-          xyz="0 0 0"
-          rpy="0 0 0" />
-        <geometry>
-          <mesh
-            filename="file://$(find rov_ricketts_description)/meshes/decal.dae" scale="1.0 1.0 1.0"/>
-        </geometry>
-        <material name="logo">
-          <texture filename="file://$(find rov_ricketts_description)/textures/logo.png"/>
-        </material>
-      </visual>
-      <collision>
-        <origin
-          xyz="0 0 0"
-          rpy="0 0 0" />
-        <geometry>
-          <mesh
-            filename="file://$(find rov_ricketts_description)/meshes/decal.dae" scale="1.0 1.0 1.0"/>
-        </geometry>
-      </collision> -->
+      <!-- alluminium structure frame -->
       <visual>
         <origin
-          xyz="0 0 0"
+          xyz="1.8143 -0.004215 -0.560595"
           rpy="0 0 0" />
         <geometry>
@@ -81,16 +46,8 @@
         </geometry>
       </visual>
-      <collision>
-        <origin
-          xyz="0 0 0"
-          rpy="0 0 0" />
-        <geometry>
-          <mesh
-            filename="file://$(find rov_ricketts_description)/meshes/frame.dae" scale="1.0 1.0 1.0"/>
-        </geometry>
-      </collision>
+      <!-- all 7 thrusters' case frames -->
       <visual>
         <origin
-          xyz="0 0 0"
+          xyz="1.8143 -0.004215 -0.560595"
           rpy="0 0 0" />
         <geometry>
@@ -99,16 +56,8 @@
         </geometry>
       </visual>
-      <collision>
-        <origin
-          xyz="0 0 0"
-          rpy="0 0 0" />
-        <geometry>
-          <mesh
-            filename="file://$(find rov_ricketts_description)/meshes/thrusters.dae" scale="1.0 1.0 1.0"/>
-        </geometry>
-      </collision>
+      <!-- internal equipment frame -->
       <visual>
         <origin
-          xyz="0 0 0"
+          xyz="1.8143 -0.004215 -0.560595"
           rpy="0 0 0" />
         <geometry>
@@ -117,42 +66,44 @@
         </geometry>
       </visual>
+      <!-- simple box collision model -->
       <collision>
         <origin
-          xyz="0 0 0"
+          xyz="0 0 -0.3"
           rpy="0 0 0" />
         <geometry>
-          <mesh
-            filename="file://$(find rov_ricketts_description)/meshes/equipment.dae" scale="1.0 1.0 1.0"/>
+             <box size="3.5 1.90 2.0"/>
         </geometry>
       </collision>
     </link>
+    <!-- dummy link -->
     <joint name="base_link_frame" type="fixed">
-      <origin rpy="0 0 0" xyz="0 0 0"/>
+      <origin rpy="0 0 0" xyz="1.8143 -0.004215 -0.560595"/>
       <parent link="base_link" />
       <child link="base_frame" />
     </joint>
     <link name="base_frame">
-      <!-- <inertial>
+    </link>
+    <joint name="base_sonar_frame" type="fixed">
+      <origin rpy="0 0 0" xyz="1.54601 -0.004325 0.730815"/>
+      <parent link="base_link" />
+      <child link="sonar_frame" />
+    </joint>
+    <link name="sonar_frame">
+    <!-- dummy inertial values for gazebo-->
+      <inertial>
         <origin
-          xyz="-1.81450712  0.00636514  0.5734822"
+          xyz="0 0 0"
           rpy="0 0 0" />
         <mass
-          value="4700.0" />
+          value="0.00000001" />
         <inertia
-          ixx="2779.72167757"
-          ixy="-142.69321245"
-          ixz="-59.10699454"
-          iyy="4409.88731132"
-          iyz="31.89417598"
-          izz="4961.49762669" />
-      </inertial> -->
+          ixx="1e-12"
+          ixy="0"
+          ixz="0"
+          iyy="1e-12"
+          iyz="0"
+          izz="1e-12" />
+      </inertial>
     </link>
-<!--
-    <joint name="base_sonar_joint" type="fixed">
-      <origin rpy="0 0 0"
-              xyz="-0.26829 -0.00011 1.29141"/>
-      <parent link="base_link" />
-      <child link="sonar_link" />
-    </joint> -->
   </xacro:macro>
 </robot>

File: rov_ricketts_description/urdf/joint_states_publisher_plugin.xacro (robot description, xacro)
@@ -1,9 +1,8 @@
 <?xml version="1.0"?>
 <robot xmlns:xacro="http://ros.org/wiki/xacro">
-    <xacro:arg name="load_arm" default="false" />
-        <xacro:macro name="all_joint_state_macro" params="load_arm name">
-            <!-- Gazebo plugin for joint state publisher  -->
-            <gazebo>
-                <plugin name="gz::sim::systems::JointStatePublisher" filename="gz-sim-joint-state-publisher-system">
+    <xacro:macro name="joint_states_publisher_macro" params="load_arm name">
+        <!-- Gazebo plugin for joint state publisher  -->
+        <gazebo>
+            <plugin name="gz::sim::systems::JointStatePublisher" filename="gz-sim-joint-state-publisher-system">
                 <!-- <update_rate>500</update_rate> -->
                 <topic>/joint_states</topic>
@@ -26,6 +25,6 @@
                     <joint_name>${name}_link5_claw_left</joint_name>
                 </xacro:if>
-                </plugin>
-            </gazebo>
-        </xacro:macro>
+            </plugin>
+        </gazebo>
+    </xacro:macro>
 </robot>
